File: ram_bank.kicad_sch (KiCad schematic)
At the start: 8 parts, among them U1 TC518512FTL-70, U2 TC518512FTL-70, U3 TC518512FTL-70, U4 TC518512FTL-70

Commit message: various improvements
Parts:
- C1, C2, C3, C4: footprint Capacitor_SMD:C_1206_3216Metric -> Capacitor_SMD:C_1206_3216Metric_Pad1.33x1.80mm_HandSolder
- U1: footprint Package_SO:TSOP-II-32_21.0x10.2mm_P1.27mm -> RAMdemption:TSOP-II-32_Data0
- U2: footprint Package_SO:TSOP-II-32_21.0x10.2mm_P1.27mm -> RAMdemption:TSOP-II-32_ReversedAddr
- U4: footprint Package_SO:TSOP-II-32_21.0x10.2mm_P1.27mm -> RAMdemption:TSOP-II-NormalAddr-Data3
Changed lines of the file:
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@@
 			)
 		)
-		(property "Footprint" "Package_SO:TSOP-II-32_21.0x10.2mm_P1.27mm"
+		(property "Footprint" "RAMdemption:TSOP-II-32_ReversedAddr"
 			(at 122.174 57.15 0)
 			(effects
@@
 			)
 		)
-		(property "Datasheet" "https://datasheet4u.com/pdf-down/T/C/5/TC518512PL-70-Toshiba.pdf"
+		(property "Datasheet" ""
 			(at 126.746 128.778 0)
 			(effects
@@
 			)
 		)
-		(property "Description" "512K x 8 Pseudo-SRAM, 70 ns, TSOP-II-32"
+		(property "Description" ""
 			(at 120.65 54.102 0)
 			(effects
@@
 			)
 		)
-		(property "Footprint" "Capacitor_SMD:C_1206_3216Metric"
+		(property "Footprint" "Capacitor_SMD:C_1206_3216Metric_Pad1.33x1.80mm_HandSolder"
 			(at 141.2748 31.75 0)
 			(effects
@@
 			)
 		)
-		(property "Footprint" "Package_SO:TSOP-II-32_21.0x10.2mm_P1.27mm"
+		(property "Footprint" "RAMdemption:TSOP-II-32_Data0"
 			(at 58.674 57.15 0)
 			(effects
@@
 			)
 		)
-		(property "Datasheet" "https://datasheet4u.com/pdf-down/T/C/5/TC518512PL-70-Toshiba.pdf"
+		(property "Datasheet" ""
 			(at 63.246 128.778 0)
 			(effects
@@
 			)
 		)
-		(property "Description" "512K x 8 Pseudo-SRAM, 70 ns, TSOP-II-32"
+		(property "Description" ""
 			(at 57.15 54.102 0)
 			(effects
@@
 			)
 		)
-		(property "Footprint" "Capacitor_SMD:C_1206_3216Metric"
+		(property "Footprint" "Capacitor_SMD:C_1206_3216Metric_Pad1.33x1.80mm_HandSolder"
 			(at 153.9748 31.75 0)
 			(effects
@@
 			)
 		)
-		(property "Footprint" "Capacitor_SMD:C_1206_3216Metric"
+		(property "Footprint" "Capacitor_SMD:C_1206_3216Metric_Pad1.33x1.80mm_HandSolder"
 			(at 160.3248 31.75 0)
 			(effects
@@
 			)
 		)
-		(property "Footprint" "Capacitor_SMD:C_1206_3216Metric"
+		(property "Footprint" "Capacitor_SMD:C_1206_3216Metric_Pad1.33x1.80mm_HandSolder"
 			(at 147.6248 31.75 0)
 			(effects
@@
 			)
 		)
-		(property "Footprint" "Package_SO:TSOP-II-32_21.0x10.2mm_P1.27mm"
+		(property "Footprint" "RAMdemption:TSOP-II-NormalAddr-Data3"
 			(at 249.174 57.15 0)
 			(effects
@@
 			)
 		)
-		(property "Datasheet" "https://datasheet4u.com/pdf-down/T/C/5/TC518512PL-70-Toshiba.pdf"
+		(property "Datasheet" ""
 			(at 253.746 128.778 0)
 			(effects
@@
 			)
 		)
-		(property "Description" "512K x 8 Pseudo-SRAM, 70 ns, TSOP-II-32"
+		(property "Description" ""
 			(at 247.65 54.102 0)
 			(effects
