File: RAMdemption.kicad_sch (KiCad schematic)
At the start: 1 part, among them J1 Conn_RAM_Expansion

Commit message: shuffle around files
Parts:
- J1: footprint RAMdemption:TE_5-104652-7 -> RAMdemption:TE_5-104652-7_NoHoles
Changed lines of the file:
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@@
 			)
 		)
-		(property "Footprint" "RAMdemption:TE_5-104652-7"
+		(property "Footprint" "RAMdemption:TE_5-104652-7_NoHoles"
 			(at 48.26 95.25 0)
 			(effects

Commit message: fix drc
Other:
- sheet RAM Bank 1: file ram_bank.kicad_sch -> ram_bank_1.kicad_sch
- sheet RAM Bank 2: file ram_bank.kicad_sch -> ram_bank_2.kicad_sch
- sheet RAM Bank 3: file ram_bank.kicad_sch -> ram_bank_3.kicad_sch
- sheet RAM Bank 4: file ram_bank.kicad_sch -> ram_bank_4.kicad_sch
- sheet RAM Bank 5: file ram_bank.kicad_sch -> ram_bank_5.kicad_sch
Changed lines of the file:
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@@
 			)
 		)
-		(property "Sheetfile" "ram_bank.kicad_sch"
+		(property "Sheetfile" "ram_bank_1.kicad_sch"
 			(at 99.06 46.3046 0)
 			(effects
@@
 			)
 		)
-		(property "Sheetfile" "ram_bank.kicad_sch"
+		(property "Sheetfile" "ram_bank_4.kicad_sch"
 			(at 99.06 122.5046 0)
 			(effects
@@
 			)
 		)
-		(property "Sheetfile" "ram_bank.kicad_sch"
+		(property "Sheetfile" "ram_bank_2.kicad_sch"
 			(at 99.06 71.7046 0)
 			(effects
@@
 			)
 		)
-		(property "Sheetfile" "ram_bank.kicad_sch"
+		(property "Sheetfile" "ram_bank_5.kicad_sch"
 			(at 99.06 147.9046 0)
 			(effects
@@
 			)
 		)
-		(property "Sheetfile" "ram_bank.kicad_sch"
+		(property "Sheetfile" "ram_bank_3.kicad_sch"
 			(at 99.06 97.1046 0)
 			(effects
