File: RAMdemption.kicad_pcb (KiCad board)
At the start: 6 copper layers, 99 x 53.5 mm, 42 parts, among them J1 Conn_RAM_Expansion, U1 TC518512FTL-70, U10 TC518512FTL-70, U11 TC518512FTL-70, U12 TC518512FTL-70, U13 TC518512FTL-70, U14 TC518512FTL-70, U15 TC518512FTL-70, U16 TC518512FTL-70, U17 TC518512FTL-70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

Commit message: pcb page size
Parts:
- moved C11 73.4 mm to (182.8, 121.0)
- moved C14 73.4 mm to (182.8, 111.4)
- moved C15 73.4 mm to (159.4, 105.9)
- moved C17 73.4 mm to (107.2, 111.3)
- moved C19 73.4 mm to (159.6, 94.3)
- moved C2 73.4 mm to (182.5, 81.3)
- moved C20 73.4 mm to (157.1, 94.2)
- moved C3 73.4 mm to (159.6, 94.3)
- moved C4 73.4 mm to (157.1, 94.2)
- moved C6 73.4 mm to (182.8, 111.4)
- moved C8 73.4 mm to (144.9, 121.9)
- moved U10 73.4 mm to (194.3, 116.3)
- moved U12 73.4 mm to (149.7, 110.1)
- moved U14 73.4 mm to (194.3, 101.1)
- moved U18 73.4 mm to (194.3, 86.1)
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
Commit message: prepare for production
Parts:
- moved C11 23.5 mm to (159.3, 121.0)
- moved C10 23.5 mm to (182.7, 121.0)
Routing:
- net /~{WE1}: track 44.3 -> 45.7 mm
